File: hardware/rover回路_試作/raspberryPi.sch (KiCad schematic (older format))
At the start: 1 part

Commit message: rover回路最終版v1.0 降圧回路に関してのみ未記載
Parts:
- added D?: LED, symbol Device:LED
- added R?: R, symbol Device:R
- added SW?: SW_DPDT_x2, symbol Switch:SW_DPDT_x2
Connections:
- net labels added: +5V, 5V_GND, 5V_typeC, PICO_QUICK, WALLPOST, WALL_FRONT, WALL_LEFt, WALL_RIGHT
- net labels removed: +3.3V, GND, GPIO_X, powerUSB
- wire segments 18 -> 36
